File: Board/Robot Controller PCB/Robot Controller PCB.kicad_pcb (KiCad board)
At the start: 2 copper layers, 96.5 x 40.6 mm, 17 parts, among them SW1 SW_DIP_x04, SW2 SW_Push, SW3 SW_Push, U1 Sparkfun_Pro_Micro

Commit message: Done....for now
Parts:
- Arduino Leonardo : renamed from U1
- gnd, led, push: renamed from sw_led1
- gnd, led, push: renamed from sw_led4
- gnd, led, push: renamed from sw_led2
- gnd, led, push: renamed from sw_led3
- gnd, vcc, dtb: renamed from VR3
- gnd, vcc, dtb: renamed from VR2
- gnd, vcc, dtb: renamed from VR1
- gnd, vcc, dtb: renamed from VR4
- moved gnd, led, push 12.7 mm to (152.4, 96.5)
- moved R1(10k) 10.2 mm to (94.0, 119.4), turned to -90 degrees
- moved gnd, led, push 7.62 mm to (142.2, 96.5)
- renumbered SW1 to Dipswitch, R1 to R1(10k), R2 to R2(20k), R3 to R3(40k), R4 to R4(80k), R5 to R5(10k), SW2 to Toggle, SW3 to Toggle
Connections:
- gnd, led, push pad 1: Net-(U1-Pad13) -> Net-(U1-Pad11)
- gnd, led, push pad 2: Net-(U1-Pad9) -> Net-(U1-Pad15)
- gnd, led, push pad 1: Net-(U1-Pad14) -> Net-(U1-Pad9)
- gnd, led, push pad 2: Net-(U1-Pad11) -> Net-(U1-Pad10)
- gnd, led, push pad 1: Net-(U1-Pad15) -> Net-(U1-Pad14)
- gnd, led, push pad 2: Net-(U1-Pad10) -> Net-(U1-Pad13)
Routing:
- net Net-(R1-Pad1): track 0.00 -> 53.7 mm
- net Net-(SW3-Pad2): track 0.00 -> 45.4 mm
- net Net-(SW2-Pad2): track 0.00 -> 41.8 mm
- net Net-(U1-Pad20): track 0.00 -> 34.6 mm
- net Net-(R4-Pad1): track 0.00 -> 34.1 mm
- net Net-(U1-Pad19): track 0.00 -> 28.8 mm
- net Net-(U1-Pad17): track 0.00 -> 27.6 mm
- net Net-(R3-Pad1): track 0.00 -> 25.5 mm
- net Net-(R2-Pad1): track 0.00 -> 17.5 mm
- net Net-(U1-Pad18): track 0.00 -> 16.4 mm
- net Net-(U1-Pad9): track 45.3 -> 29.7 mm
- net Net-(U1-Pad11): track 31.9 -> 45.7 mm
- net Net-(U1-Pad13): track 51.3 -> 39.4 mm
- net +5V: track 0.00 -> 10.2 mm
- net Net-(U1-Pad16): track 39.8 -> 29.8 mm
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- added copper zone on F.Cu, net +5V
- added copper zone on B.Cu, net GND
Other:
- outline, holes or cut-outs redrawn
- board text added: "Button"
- board text added: "Code, PCB, CAD, and other recorces:"
- board text added: "Created by Chris Spooner and Noah Clark"
- board text added: "Main Brain"
- board text added: "Momentary"
- board text added: "Slider"
- board text added: "Toggle"
- board text added: "https://github.com/cspoonerKRHS/RobotController"
